File: esquematico_kicad/esquematico_kicad.sch (KiCad schematic (older format))
At the start: 2 parts

Commit message: update
Parts:
- removed U?: ESP32, ESP32-footprints-Lib:ESP32, symbol ESP32:ESP32
- removed U?: FT232RL, Package_SO:SSOP-28_5.3x10.2mm_P0.65mm, symbol Interface_USB:FT232RL
- added J?: Conn_01x04_Female, symbol Connector:Conn_01x04_Female
- added U?: ESP32-WROOM-32D, RF_Module:ESP32-WROOM-32, symbol RF_Module:ESP32-WROOM-32D
Connections:
- new net: U?.1 (GND), U?.15 (GND), U?.38 (GND), U?.39 (GND)
Changed lines of the file:
@@
 $Descr A4 11693 8268
 encoding utf-8
-Sheet 1 1
+Sheet 1 2
 Title ""
 Date ""
@@
 $EndDescr
 $Comp
-L ESP32:ESP32 U?
-U 1 1 618D2927
-P 6000 3900
-F 0 "U?" H 6000 5737 60  0000 C CNN
-F 1 "ESP32" H 6000 5631 60  0000 C CNN
-F 2 "ESP32-footprints-Lib:ESP32" H 6450 4800 60  0001 C CNN
-F 3 "" H 6450 4800 60  0001 C CNN
-	1    6000 3900
+L Connector:Conn_01x04_Female J?
+U 1 1 61942D89
+P 8500 3050
+F 0 "J?" H 8528 3026 50  0000 L CNN
+F 1 "Conn_01x04_Female" H 8528 2935 50  0000 L CNN
+F 2 "" H 8500 3050 50  0001 C CNN
+F 3 "~" H 8500 3050 50  0001 C CNN
+	1    8500 3050
 	1    0    0    -1
 $EndComp
-Wire Wire Line
-	3050 3050 3900 3050
-Wire Wire Line
-	3900 3050 3900 5000
-Wire Wire Line
-	3900 5000 5150 5000
-Wire Wire Line
-	3050 3150 3800 3150
-Wire Wire Line
-	3800 3150 3800 5100
-Wire Wire Line
-	3800 5100 5150 5100
-Wire Wire Line
-	3050 3350 3650 3350
-Wire Wire Line
-	3650 3350 3650 5750
-Wire Wire Line
-	3650 5750 7000 5750
-Wire Wire Line
-	7000 5750 7000 4050
-Wire Wire Line
-	7000 4050 6850 4050
-Wire Wire Line
-	3050 3250 3750 3250
-Wire Wire Line
-	3750 3250 3750 5600
-Wire Wire Line
-	3750 5600 6900 5600
-Wire Wire Line
-	6900 5600 6900 4250
-Wire Wire Line
-	6900 4250 6850 4250
+$Sheet
+S 3150 1650 1400 650
+U 61943D7C
+F0 "Sheet61943D7B" 50
+F1 "alimentacion.sch" 50
+$EndSheet
 $Comp
-L Interface_USB:FT232RL U?
-U 1 1 618D5DB8
-P 2250 3750
-F 0 "U?" H 2250 4931 50  0000 C CNN
-F 1 "FT232RL" H 2250 4840 50  0000 C CNN
-F 2 "Package_SO:SSOP-28_5.3x10.2mm_P0.65mm" H 3350 2850 50  0001 C CNN
-F 3 "https://www.ftdichip.com/Support/Documents/DataSheets/ICs/DS_FT232R.pdf" H 2250 3750 50  0001 C CNN
-	1    2250 3750
+L RF_Module:ESP32-WROOM-32D U?
+U 1 1 619769EC
+P 5900 3400
+F 0 "U?" H 5900 4981 50  0000 C CNN
+F 1 "ESP32-WROOM-32D" H 5900 4890 50  0000 C CNN
+F 2 "RF_Module:ESP32-WROOM-32" H 5900 1900 50  0001 C CNN
+F 3 "https://www.espressif.com/sites/default/files/documentation/esp32-wroom-32d_esp32-wroom-32u_datasheet_en.pdf" H 5600 3450 50  0001 C CNN
+	1    5900 3400
 	1    0    0    -1
 $EndComp
