File: KiCAD - Controlador de Aforo/alimentacion.sch (KiCad schematic (older format))
At the start: 0 parts

Commit message: kicad alimentacion
Parts:
- added C?: 10uF, symbol Device:C_Small
- added C?: 100uF, symbol Device:C_Small
- added D1: GREEN, symbol Device:LED
- added D2: RED, symbol Device:LED
- added J?: BAT+, symbol Connector_Generic:Conn_01x01
- added J?: BAT-, symbol Connector_Generic:Conn_01x01
- added P?: USB_C_Plug_USB2.0, symbol Connector:USB_C_Plug_USB2.0
- added R? (x2), R_prog, R_prog?: 1K, symbol Device:R
- added R_prog?: 100, symbol Device:R
- added U?: TP4056, symbol tp4056:TP4056
- added U?: DW01, symbol dw01:DW01
- added U?: FS8205A, symbol fs8205a:FS8205A
Connections:
- new net: R_prog.1, U?.2 (PROG)
- new net: C?.1, D1.2 (A), D2.2 (A), P?.A4 (VBUS), P?.A9 (VBUS), P?.B4 (VBUS), P?.B9 (VBUS), U?.4 (VCC), U?.8 (CE)
- new net: R?.2, U?.6 (~STDBY)
- new net: R?.2, U?.7 (~CHRG)
- new net: U?.1 (OD), U?.4 (G1)
- new net: R_prog?.1, U?.2 (CS)
- new net: U?.3 (OC), U?.5 (G2)
- new net: C?.2, R_prog?.2, U?.5 (VCC)
- new net: C?.1, J?.1 (Pin_1), U?.2 (S1), U?.3 (S1), U?.6 (GND)
- new net: D1.1 (K), R?.1
- new net: D2.1 (K), R?.1
- new net Earth: C?.2, P?.A1 (GND), P?.A12 (GND), P?.B1 (GND), P?.B12 (GND), R_prog.2, R_prog?.2, U?.1 (TEMP), U?.3 (GND), U?.6 (S2), U?.7 (S2)
- new net VCC: J?.1 (Pin_1), R_prog?.1, U?.5 (BAT)
