File: KiCAD - Controlador de Aforo/alimentacion.sch (KiCad schematic (older format))
At the start: 15 parts

Commit message: software
Parts:
- added D3: D_Schottky_ALT, symbol Device:D_Schottky_ALT
- added L1: L, symbol Device:L
- gave numbers to parts that had none: 12
- renumbered R_prog to R_prog1
Changed lines of the file:
@@
 $EndDescr
 $Comp
-L tp4056:TP4056 U?
+L tp4056:TP4056 U2
 U 1 1 619D01DE
 P 5250 2250
-F 0 "U?" H 5250 2787 60  0000 C CNN
+F 0 "U2" H 5250 2787 60  0000 C CNN
 F 1 "TP4056" H 5250 2681 60  0000 C CNN
 F 2 "" H 5250 2250 60  0000 C CNN
@@
 $EndComp
 $Comp
-L dw01:DW01 U?
+L dw01:DW01 U3
 U 1 1 619D0701
 P 7650 1900
-F 0 "U?" H 7675 2337 60  0000 C CNN
+F 0 "U3" H 7675 2337 60  0000 C CNN
 F 1 "DW01" H 7675 2231 60  0000 C CNN
 F 2 "" H 7600 1600 60  0001 C CNN
@@
 $EndComp
 $Comp
-L fs8205a:FS8205A U?
+L fs8205a:FS8205A U4
 U 1 1 619D0F1A
 P 8200 3150
-F 0 "U?" V 7713 3050 60  0000 C CNN
+F 0 "U4" V 7713 3050 60  0000 C CNN
 F 1 "FS8205A" V 7819 3050 60  0000 C CNN
 F 2 "" H 9150 3400 60  0001 C CNN
@@
 $EndComp
 $Comp
-L Connector:USB_C_Plug_USB2.0 P?
+L Connector:USB_C_Plug_USB2.0 P1
 U 1 1 619D1FFE
 P 2150 2350
-F 0 "P?" H 2257 3217 50  0000 C CNN
+F 0 "P1" H 2257 3217 50  0000 C CNN
 F 1 "USB_C_Plug_USB2.0" H 2257 3126 50  0000 C CNN
 F 2 "" H 2300 2350 50  0001 C CNN
@@
 $EndComp
 $Comp
-L Device:R R?
+L Device:R R1
 U 1 1 619D4DAC
 P 3650 2400
-F 0 "R?" H 3720 2446 50  0000 L CNN
+F 0 "R1" H 3720 2446 50  0000 L CNN
 F 1 "1K" H 3720 2355 50  0000 L CNN
 F 2 "" V 3580 2400 50  0001 C CNN
@@
 $EndComp
 $Comp
-L Device:R R?
+L Device:R R2
 U 1 1 619DA812
 P 4100 2400
-F 0 "R?" H 4170 2446 50  0000 L CNN
+F 0 "R2" H 4170 2446 50  0000 L CNN
 F 1 "1K" H 4170 2355 50  0000 L CNN
 F 2 "" V 4030 2400 50  0001 C CNN
@@
 	4600 2000 4600 2100
 $Comp
-L power:Earth #PWR?
+L power:Earth #PWR02
 U 1 1 619E35EA
 P 3200 3050
-F 0 "#PWR?" H 3200 2800 50  0001 C CNN
+F 0 "#PWR02" H 3200 2800 50  0001 C CNN
 F 1 "Earth" H 3200 2900 50  0001 C CNN
 F 2 "" H 3200 3050 50  0001 C CNN
@@
 	4100 1750 4600 1750
 $Comp
-L Device:C_Small C?
+L Device:C_Small C1
 U 1 1 619E7BF4
 P 3200 2400
-F 0 "C?" H 3292 2446 50  0000 L CNN
+F 0 "C1" H 3292 2446 50  0000 L CNN
 F 1 "10uF" H 3292 2355 50  0000 L CNN
 F 2 "" H 3200 2400 50  0001 C CNN
@@
 	3200 1750 3650 1750
 $Comp
-L Device:R R_prog
+L Device:R R_prog1
 U 1 1 619EC7BF
 P 6050 2800
-F 0 "R_prog" H 6120 2846 50  0000 L CNN
+F 0 "R_prog1" H 6120 2846 50  0000 L CNN
 F 1 "1K" H 6120 2755 50  0000 L CNN
 F 2 "" V 5980 2800 50  0001 C CNN
@@
 $EndComp
 $Comp
-L power:Earth #PWR?
+L power:Earth #PWR04
 U 1 1 619EDFAD
 P 6050 3050
-F 0 "#PWR?" H 6050 2800 50  0001 C CNN
+F 0 "#PWR04" H 6050 2800 50  0001 C CNN
 F 1 "Earth" H 6050 2900 50  0001 C CNN
 F 2 "" H 6050 3050 50  0001 C CNN
@@
 $EndComp
 $Comp
-L power:Earth #PWR?
+L power:Earth #PWR03
 U 1 1 619F0468
 P 5250 2750
-F 0 "#PWR?" H 5250 2500 50  0001 C CNN
+F 0 "#PWR03" H 5250 2500 50  0001 C CNN
 F 1 "Earth" H 5250 2600 50  0001 C CNN
 F 2 "" H 5250 2750 50  0001 C CNN
@@
 	5750 2400 6050 2400
 $Comp
-L Device:R R_prog?
+L Device:R R_prog2
 U 1 1 61A07F74
 P 6900 2400
-F 0 "R_prog?" H 6970 2446 50  0000 L CNN
+F 0 "R_prog2" H 6970 2446 50  0000 L CNN
 F 1 "1K" H 6970 2355 50  0000 L CNN
 F 2 "" V 6830 2400 50  0001 C CNN
@@
 	6900 3250 7500 3250
 $Comp
-L power:Earth #PWR?
+L power:Earth #PWR05
 U 1 1 61A0C11F
 P 6900 3350
-F 0 "#PWR?" H 6900 3100 50  0001 C CNN
+F 0 "#PWR05" H 6900 3100 50  0001 C CNN
 F 1 "Earth" H 6900 3200 50  0001 C CNN
 F 2 "" H 6900 3350 50  0001 C CNN
@@
 	8700 3150 8700 3250
 $Comp
-L Device:C_Small C?
+L Device:C_Small C2
 U 1 1 61A0FC38
 P 8500 1750
-F 0 "C?" V 8271 1750 50  0000 C CNN
+F 0 "C2" V 8271 1750 50  0000 C CNN
 F 1 "100uF" V 8362 1750 50  0000 C CNN
 F 2 "" H 8500 1750 50  0001 C CNN
@@
 Connection ~ 8750 1950
 $Comp
-L Device:R R_prog?
+L Device:R R_prog3
 U 1 1 61A14133
 P 8500 2200
-F 0 "R_prog?" V 8293 2200 50  0000 C CNN
+F 0 "R_prog3" V 8293 2200 50  0000 C CNN
 F 1 "100" V 8384 2200 50  0000 C CNN
 F 2 "" V 8430 2200 50  0001 C CNN
@@
 $EndComp
 $Comp
-L Connector_Generic:Conn_01x01 J?
+L Connector_Generic:Conn_01x01 J4
 U 1 1 619FA0CA
 P 9850 2650
-F 0 "J?" H 9930 2692 50  0000 L CNN
+F 0 "J4" H 9930 2692 50  0000 L CNN
 F 1 "BAT-" H 9930 2601 50  0000 L CNN
 F 2 "" H 9850 2650 50  0001 C CNN
@@
 $EndComp
 $Comp
-L Connector_Generic:Conn_01x01 J?
+L Connector_Generic:Conn_01x01 J3
 U 1 1 619F7077
 P 9850 1900
-F 0 "J?" H 9930 1942 50  0000 L CNN
+F 0 "J3" H 9930 1942 50  0000 L CNN
 F 1 "BAT+" H 9930 1851 50  0000 L CNN
 F 2 "" H 9850 1900 50  0001 C CNN
@@
 	5250 2750 5250 2650
 $Comp
-L power:Earth #PWR?
+L power:Earth #PWR01
 U 1 1 61A22222
 P 2150 3350
-F 0 "#PWR?" H 2150 3100 50  0001 C CNN
+F 0 "#PWR01" H 2150 3100 50  0001 C CNN
 F 1 "Earth" H 2150 3200 50  0001 C CNN
 F 2 "" H 2150 3350 50  0001 C CNN
@@
 	8950 1200 9300 1200
 Connection ~ 8950 1350
+Text HLabel 1800 4550 0    50   Output ~ 0
+Bat_pos
+$Comp
+L Device:L L1
+U 1 1 619FA05B
+P 2500 4250
+F 0 "L1" V 2319 4250 50  0000 C CNN
+F 1 "L" V 2410 4250 50  0000 C CNN
+F 2 "" H 2500 4250 50  0001 C CNN
+F 3 "~" H 2500 4250 50  0001 C CNN
+	1    2500 4250
+	0    1    1    0
+$EndComp
+$Comp
+L Device:D_Schottky_ALT D3
+U 1 1 619FAFDB
+P 3200 4250
+F 0 "D3" H 3200 4034 50  0000 C CNN
+F 1 "D_Schottky_ALT" H 3200 4125 50  0000 C CNN
+F 2 "" H 3200 4250 50  0001 C CNN
+F 3 "~" H 3200 4250 50  0001 C CNN
+	1    3200 4250
+	-1   0    0    1
+$EndComp
 $EndSCHEMATC
